File: ESP32-S3 Pico D1.kicad_pcb (KiCad board)
At the start: 6 copper layers, 31 x 63.5 mm, 203 parts, among them CN301 SM32B-NSHDZS-1-TF, CN302 SM32B-NSHDZS-1-TF, CN501 GT-USB-7014D, Q901 NTLJS17D0P03P8Z, SW601 SPST-NO, SW602 SPST-NO, U1001 74LV1T125, U1002 74LV1T125, U1003 74LV1T125, U1004 74LV1T125, U1005 74LV1T125, U401 ESP32-S3-PICO-1-N8R2, U501 TPS2121, U502 TPSM82903, U701 TCAN4550-Q1, U702 74LVC1G14, U801 74LV1T125, U802 74LV1T125, U803 74LV1T125, U804 74LV1T125, U805 74LV1T125, U901 74LV1T125, U902 74LV1T125, U903 TPS2HCS10A-Q1, U904 74LV1T125, U905 74LV1T125, U906 74LV1T125, U907 74LV1T125, Y701 40MHz

Commit message: Update CAN_Interface.kicad_sch, ESP32-S3 D1 Pico Board.kicad_sch, ESP32-S3 Pico D1.kicad_pcb, and 5 more files
Parts:
- removed C1001, C702, C703, C705, C713, C714, C715, C716, C801, C802, C803, C804, C805, C806, C807, C808, C809, C810, C901, C902, C903, C904, C905, C907, C908, C909, C911, C912, C913, C914: 0.1uF, My Capacitors:C_0201_Dense
- removed C701, C704, C706, C707, C708, C709, C710: 22uF, My Capacitors:C_0603_Dense
- removed C711, C712: 10pF, My Capacitors:C_0201_Dense
- removed C910, C915: 4.7nF, My Capacitors:C_0201_Dense
- removed CMC701: CMC 0805, Personal_FootprintLibrary:CMC_0805
- removed CN301, CN302: SM32B-NSHDZS-1-TF, My Connectors:JST_NSHD_SM32B-NSHD_2x16_P1.0mm_Horizontal_SMD
- removed D1001, D1002, D701, D801, D803, D804, D806, D807, D809, D810, D812, D813, D901, D902, D903, D904, D908, D909, D912, D913, D914: PMEG4002ESFYL, Personal_FootprintLibrary:DSN0603-2
- removed D702, D703: SZESD7241N2T5G, Personal_FootprintLibrary:DFN1006-2
- removed D704, D802, D805, D808, D811, D814, D905, D906, D907, D910, D911, D915, D916: D15V0H1U2LP-7B, Personal_FootprintLibrary:DFN1006-2
- removed H301, H302: ESP_Header, My Connectors:PinHeader_2x10_P2.54mm_Vertical_THT_BottomMount_TopReference
- removed Q901: NTLJS17D0P03P8Z, My Package_Leadless:WDFN6-4_2.05x2.05mm_P0.65mm
- removed R1001, R1005, R1006, R701, R805, R904, R905, R907, R908, R912, R913, R914, R917, R918: 5k1, My Resistors:R_0201_Dense
- removed R1002, R1003, R1004, R702, R901, R902, R903, R906, R910, R911, R915, R916: 33R, My Resistors:R_0201_Dense
- removed R703, R806: 470R, My Resistors:R_0201_Dense
- removed R801, R802, R803, R804: 26k1, My Resistors:R_0201_Dense
- removed R909: 100k, My Resistors:R_0201_Dense
- removed U1001, U1002, U1003, U1004, U1005, U801, U802, U803, U804, U805, U901, U902, U904, U905, U906, U907: 74LV1T125, Personal_FootprintLibrary:X2SON5_SOT1226_0.8x0.8mm
- removed U701: TCAN4550-Q1, Package_DFN_QFN:Texas_RGY_R-PVQFN-N20_EP2.05x3.05mm
- removed U702: 74LVC1G14, Personal_FootprintLibrary:X2SON5_SOT1226_0.8x0.8mm
- removed U903: TPS2HCS10A-Q1, My Package_SO:Texas_HTSSOP-16-1EP_5.0x4.4mm_P0.65mm_EP5.0x3.4mm_Mask3.313x2.78mm
- removed Y701: 40MHz, Crystal:Crystal_SMD_2016-4Pin_2.0x1.6mm
- added R406: 33R, My Resistors:R_0201_Dense, F.Cu at (154.9, 112.6)
- added R407: 33R, My Resistors:R_0201_Dense, F.Cu at (157.6, 111.4)
- added R408: 33R, My Resistors:R_0201_Dense, F.Cu at (157.6, 112.7)
Connections:
- net /ESP32-S3 Board/EN/Reset renamed /ESP32-S3 Board/EN/~{Reset}
- U401 pad 27: /ESP32-S3 Board/IO21 -> /ESP32-S3 Board/ESP32-S3-PICO-1/GPIO21
- U401 pad 36: /ESP32-S3 Board/IO48 -> Net-(U401-SPICLK_N/GPIO48)
- U401 pad 37: /ESP32-S3 Board/IO47 -> Net-(U401-SPICLK_P/GPIO47)
Routing:
- net /IO_Board/~{FAULT_{BUS}}: track 18.6 -> 0.00 mm, vias 2 -> 0
- net /IO_Board/RLY-: track 15.6 -> 0.00 mm
- net /IO_Board/RLY+: track 8.10 -> 0.00 mm
- net +5V_{FUSED}: track 23.7 -> 16.2 mm, vias 20 -> 10
- net /IO_Board/~{CS_{HSS}}: track 7.03 -> 0.00 mm, vias 2 -> 0
- net /IO_Board/~{CS_{HSS}}_{5V}: track 6.23 -> 0.00 mm
- net /ESP32-S3 Board/IO21: track 16.1 -> 9.90 mm, vias 2 -> 0
- net /IO_Board/Unified SPI and Global Fault/~{CS}: track 5.95 -> 0.00 mm, vias 2 -> 0
- net /ESP32-S3 Board/IO48: track 9.35 -> 3.55 mm
- net /IO_Board/SCLK_{5V}: track 5.71 -> 0.00 mm, vias 2 -> 0
- net /ESP32-S3 Board/ESP32-S3-PICO-1/GPIO21: track 0.00 -> 5.60 mm, vias 0 -> 2
- net /IO_Board/SCLK: track 5.56 -> 0.00 mm
- net /ESP32-S3 Board/IO47: track 12.1 -> 6.62 mm
- net Net-(U401-SPICLK_N/GPIO48): track 0.00 -> 5.24 mm
- net Net-(U401-SPICLK_P/GPIO47): track 0.00 -> 4.95 mm
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- removed copper zone on In3.Cu, net +3V3
- removed copper zone on In4.Cu, net +5V_{FUSED}
- removed copper zone on B.Cu, net +V_{BAT}
- removed copper zone on F.Cu, net +V_{SW}
- removed copper zone on In2.Cu, net +V_{SW}
- removed copper zone on F.Cu, net /IO_Board/WLED Outputs/V_{OUT1}
- removed copper zone on In2.Cu, net /IO_Board/WLED Outputs/V_{OUT1}
- removed copper zone on F.Cu, net /IO_Board/WLED Outputs/V_{OUT2}
- removed copper zone on In2.Cu, net /IO_Board/WLED Outputs/V_{OUT2}
- removed copper zone on F.Cu, net GND2
Other:
- board size 31 x 63.5 mm -> 31 x 30.5 mm
